File: DRV8962DDWR.kicad_sch (KiCad schematic)
At the start: 10 parts, among them U1 DRV8962DDWR

Commit message: add pd power
Connections:
- net +24V renamed VBUS
Changed lines of the file:
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@@
 			)
 		)
-		(property "Value" "+24V"
+		(property "Value" "VBUS"
 			(at 166.37 57.15 0)
 			(effects

Commit message: feat: add as5047p
Connections:
- net DRV8962_VREF renamed +3.3VA
Changed lines of the file:
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@@
+	(wire
+		(pts
+			(xy 111.76 76.2) (xy 134.62 76.2)
+		)
+		(stroke
+			(width 0)
+			(type default)
+		)
+	)
 	(wire
 		(pts
@@
 	(wire
 		(pts
+			(xy 111.76 74.93) (xy 111.76 76.2)
+		)
+		(stroke
+			(width 0)
+			(type default)
+		)
+	)
+	(wire
+		(pts
 			(xy 162.56 113.03) (xy 165.1 113.03)
 		)
@@
 		(pts
 			(xy 162.56 62.23) (xy 163.83 62.23)
-		)
-		(stroke
-			(width 0)
-			(type default)
-		)
-	)
-	(wire
-		(pts
-			(xy 133.35 76.2) (xy 134.62 76.2)
 		)
 		(stroke
@@
 		(shape input)
 		(at 132.08 114.3 180)
-		(effects
-			(font
-				(size 1.27 1.27)
-			)
-			(justify right)
-		)
-	)
-	(hierarchical_label "DRV8962_VREF"
-		(shape input)
-		(at 133.35 76.2 180)
 		(effects
 			(font
@@
 					(unit 1)
 				)
+			)
+		)
+	)
+	(symbol
+		(lib_id "power:+3.3V")
+		(at 111.76 74.93 0)
+		(unit 1)
+		(exclude_from_sim no)
+		(in_bom yes)
+		(on_board yes)
+		(dnp no)
+		(property "Reference" "#PWR041"
+			(at 111.76 78.74 0)
+			(effects
+				(font
+					(size 1.27 1.27)
+				)
+				(hide yes)
+			)
+		)
+		(property "Value" "+3.3VA"
+			(at 111.76 70.866 0)
+			(effects
+				(font
+					(size 1.27 1.27)
+				)
+			)
+		)
+		(property "Footprint" ""
+			(at 111.76 74.93 0)
+			(effects
+				(font
+					(size 1.27 1.27)
+				)
+				(hide yes)
+			)
+		)
+		(property "Datasheet" ""
+			(at 111.76 74.93 0)
+			(effects
+				(font
+					(size 1.27 1.27)
+				)
+				(hide yes)
+			)
+		)
+		(property "Description" "Power symbol creates a global label with name \"+3.3V\""
+			(at 111.76 74.93 0)
+			(effects
+				(font
+					(size 1.27 1.27)
+				)
+				(hide yes)
+			)
+		)
+		(pin "1"
+		)
+		(instances
+			(project "foc-stepper-driver"
+				(path "/e8a1091a-f86c-4a0e-9f89-1944d2e62a64/a16ad1d8-3628-4dc7-b4ec-9c3a867ebe41"
+					(reference "#PWR041")
+					(unit 1)
+				)

Commit message: feat: add can and usart connector
Parts:
- C3: value 100nF -> 100n
- C4, C6, C7: value 10nF -> 10n
- C5, C8: value 1uF -> 1u
Changed lines of the file:
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@@
 			)
 		)
-		(property "Value" "10nF"
+		(property "Value" "10n"
 			(at 197.485 80.01 0)
 			(effects
@@
 			)
 		)
-		(property "Value" "1uF"
+		(property "Value" "1u"
 			(at 128.27 69.342 90)
 			(effects
@@
 			)
 		)
-		(property "Value" "1uF"
+		(property "Value" "1u"
 			(at 183.642 60.96 0)
 			(effects
@@
 			)
 		)
-		(property "Value" "10nF"
+		(property "Value" "10n"
 			(at 205.105 80.01 0)
 			(effects
@@
 			)
 		)
-		(property "Value" "100nF"
+		(property "Value" "100n"
 			(at 123.19 55.8799 0)
 			(effects
@@
 			)
 		)
-		(property "Value" "10nF"
+		(property "Value" "10n"
 			(at 189.865 80.01 0)
 			(effects

Commit message: change components
Parts:
- added C20: 47u, Capacitor_SMD:C_0402_1005Metric, symbol Device:C_Small_US
- added C21: 10n, Capacitor_SMD:C_0402_1005Metric, symbol Device:C
- C3, C4, C5, C6, C7, C8: footprint (none) -> Capacitor_SMD:C_0402_1005Metric
- R1, R2, R3: footprint (none) -> PCM_Resistor_SMD_AKL:R_0402_1005Metric
Connections:
- net GND: now also C20.1, C21.2
- net VBUS renamed +24V
- net +24V: now also C20.2, C21.1
Other:
- note added: "50V, 10nF ceramic capacitor"
- note added: "50V, 47uF bulk capacitor"
- note added: "Max Current: 5A"
- note added: "Motor Driver and Currnet Sensing"
- moved on the sheet: C4, C6, C7

Commit message: update sch
Other:
- moved on the sheet: C8
Changed lines of the file:
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@@
 	(wire
 		(pts
-			(xy 111.76 76.2) (xy 134.62 76.2)
+			(xy 102.87 76.2) (xy 134.62 76.2)
 		)
 		(stroke
@@
 	(wire
 		(pts
+			(xy 110.49 72.39) (xy 110.49 69.85)
+		)
+		(stroke
+			(width 0)
+			(type default)
+		)
+	)
+	(wire
+		(pts
 			(xy 133.35 99.06) (xy 134.62 99.06)
 		)
@@
 	(wire
 		(pts
-			(xy 111.76 74.93) (xy 111.76 76.2)
+			(xy 102.87 74.93) (xy 102.87 76.2)
 		)
 		(stroke
@@
 	(wire
 		(pts
-			(xy 131.572 71.374) (xy 128.778 71.374)
+			(xy 131.572 72.39) (xy 128.27 72.39)
+		)
+		(stroke
+			(width 0)
+			(type default)
+		)
+	)
+	(wire
+		(pts
+			(xy 110.49 72.39) (xy 120.65 72.39)
 		)
 		(stroke
@@
 	(wire
 		(pts
-			(xy 117.602 71.374) (xy 121.158 71.374)
-		)
-		(stroke
-			(width 0)
-			(type default)
-		)
-	)
-	(wire
-		(pts
 			(xy 132.08 114.3) (xy 134.62 114.3)
 		)
@@
 	(wire
 		(pts
-			(xy 131.572 73.66) (xy 131.572 71.374)
+			(xy 131.572 73.66) (xy 131.572 72.39)
 		)
 		(stroke
@@
 			(width 0)
 			(type default)
-		)
-	)
-	(label "VM"
-		(at 117.856 71.374 0)
-		(effects
-			(font
-				(size 1.27 1.27)
-			)
-			(justify left bottom)
 		)
 	)
@@
 	(label "DRV8962_DVDD"
 		(at 165.735 54.61 0)
-		(effects
-			(font
-				(size 1.27 1.27)
-			)
-			(justify left bottom)
-		)
-	)
-	(label "VM"
-		(at 168.91 72.39 0)
 		(effects
 			(font
@@
 	)
 	(symbol
+		(lib_id "power:+24V")
+		(at 110.49 69.85 0)
+		(mirror y)
+		(unit 1)
+		(exclude_from_sim no)
+		(in_bom yes)
+		(on_board yes)
+		(dnp no)
+		(property "Reference" "#PWR04"
+			(at 110.49 73.66 0)
+			(effects
+				(font
+					(size 1.27 1.27)
+				)
+				(hide yes)
+			)
+		)
+		(property "Value" "+24V"
+			(at 110.49 66.04 0)
+			(effects
+				(font
+					(size 1.27 1.27)
+				)
+			)
+		)
+		(property "Footprint" ""
+			(at 110.49 69.85 0)
+			(effects
+				(font
+					(size 1.27 1.27)
+				)
+				(hide yes)
+			)
+		)
+		(property "Datasheet" ""
+			(at 110.49 69.85 0)
+			(effects
+				(font
+					(size 1.27 1.27)
+				)
+				(hide yes)
+			)
+		)
+		(property "Description" "Power symbol creates a global label with name \"+24V\""
+			(at 110.49 69.85 0)
+			(effects
+				(font
+					(size 1.27 1.27)
+				)
+				(hide yes)
+			)
+		)
+		(pin "1"
+		)
+		(instances
+			(project "foc-stepper-driver"
+				(path "/e8a1091a-f86c-4a0e-9f89-1944d2e62a64/a16ad1d8-3628-4dc7-b4ec-9c3a867ebe41"
+					(reference "#PWR04")
+					(unit 1)
+				)
+			)
+		)
+	)
+	(symbol
 		(lib_id "Device:R")
 		(at 125.73 135.89 0)
@@
 	(symbol
 		(lib_id "Device:C")
-		(at 124.968 71.374 90)
+		(at 124.46 72.39 90)
 		(unit 1)
 		(exclude_from_sim no)
@@
 		(dnp no)
 		(property "Reference" "C8"
-			(at 122.174 69.342 90)
+			(at 121.666 70.358 90)
 			(effects
 				(font
@@
 		)
 		(property "Value" "1u"
-			(at 128.27 69.342 90)
+			(at 127.762 70.358 90)
 			(effects
 				(font
@@
 		)
 		(property "Footprint" "Capacitor_SMD:C_0402_1005Metric"
-			(at 128.778 70.4088 0)
+			(at 128.27 71.4248 0)
 			(effects
 				(font
@@
 		)
 		(property "Datasheet" "~"
-			(at 124.968 71.374 0)
+			(at 124.46 72.39 0)
 			(effects
 				(font
@@
 		)
 		(property "Description" "Unpolarized capacitor"
-			(at 124.968 71.374 0)
+			(at 124.46 72.39 0)
 			(effects
 				(font
@@
 	(symbol
 		(lib_id "power:+3.3V")
-		(at 111.76 74.93 0)
+		(at 102.87 74.93 0)
 		(unit 1)
 		(exclude_from_sim no)
@@
 		(dnp no)
 		(property "Reference" "#PWR041"
-			(at 111.76 78.74 0)
+			(at 102.87 78.74 0)
 			(effects
 				(font
@@
 		)
 		(property "Value" "+3.3VA"
-			(at 111.76 70.866 0)
+			(at 102.87 70.866 0)
 			(effects
 				(font
@@
 		)
 		(property "Footprint" ""
-			(at 111.76 74.93 0)
+			(at 102.87 74.93 0)
 			(effects
 				(font
@@
 		)
 		(property "Datasheet" ""
-			(at 111.76 74.93 0)
+			(at 102.87 74.93 0)
 			(effects
 				(font
@@
 		)
 		(property "Description" "Power symbol creates a global label with name \"+3.3V\""
-			(at 111.76 74.93 0)
-			(effects
-				(font
+			(at 102.87 74.93 0)
+			(effects
+				(font
