File: DRV8962DDWR.kicad_sch (KiCad schematic)
At the start: 12 parts, among them U1 DRV8962DDWR

Commit message: update
Parts:
- C13: footprint EasyEDA_Lib:CAP-SMD_BD6.3-L6.6-W6.6-LS7.3-FD -> EasyEDA_Lib:CAP-SMD_BD6.3-L6.6-W6.6-LS7.6-FD; symbol EasyEDA_Lib:RV50V47M6X5 -> EasyEDA_Lib:RVT1H470M0607; Manufacturer JIERR(捷而瑞) -> ROQANG(容强); Manufacturer Part RV50V47M6X5 -> RVT1H470M0607; Supplier Part C48971023 -> C72523
- R3: footprint PCM_Resistor_SMD_AKL:R_0402_1005Metric -> Resistor_SMD:R_0805_2012Metric
Changed lines of the file:
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@@
+	(wire
+		(pts
+			(xy 217.17 72.39) (xy 217.17 73.66)
+		)
+		(stroke
+			(width 0)
+			(type default)
+		)
+	)
 	(wire
 		(pts
@@
 		(pts
 			(xy 116.84 140.97) (xy 116.84 142.24)
+		)
+		(stroke
+			(width 0)
+			(type default)
+		)
+	)
+	(wire
+		(pts
+			(xy 217.17 81.28) (xy 217.17 82.55)
 		)
 		(stroke
@@
 			)
 		)
-		(property "Footprint" "PCM_Resistor_SMD_AKL:R_0402_1005Metric"
+		(property "Footprint" "Resistor_SMD:R_0805_2012Metric"
 			(at 106.172 58.42 90)
 			(effects
@@
 	)
 	(symbol
-		(lib_id "EasyEDA_Lib:RV50V47M6X5")
+		(lib_id "EasyEDA_Lib:RVT1H470M0607")
 		(at 217.17 77.47 270)
 		(unit 1)
@@
 			)
 		)
-		(property "Footprint" "EasyEDA_Lib:CAP-SMD_BD6.3-L6.6-W6.6-LS7.3-FD"
+		(property "Footprint" "EasyEDA_Lib:CAP-SMD_BD6.3-L6.6-W6.6-LS7.6-FD"
 			(at 217.17 77.47 0)
 			(effects
@@
 			)
 		)
-		(property "Datasheet" "https://item.szlcsc.com/datasheet/RV50V47M6X5/51296228.html"
+		(property "Datasheet" "https://item.szlcsc.com/datasheet/RVT1H470M0607/73634.html"
 			(at 217.17 77.47 0)
 			(effects
@@
 			)
 		)
-		(property "Description" "Capacitance:47uF Tolerance:±20% Tolerance:±20% Voltage Rating:50V Ripple Current:50mA@120Hz Diameter:6.3mm Height - Seated (Max):5.4mm Lifetime:2000hrs@105°C Operating Temperature:-40°C~+105°C Operating Temperature:-40°C~+105°C"
+		(property "Description" "Capacitance:47uF Tolerance:±20% Tolerance:±20% Voltage Rating:50V Ripple Current:66mA@120Hz Equivalent Series Resistance(ESR):- Diameter:6.3mm Height - Seated (Max):7.7mm Lifetime:2000hrs@105°C Operating Temperature:-40°C~+105°C Operating Temperature:-40°C~+1"
 			(at 217.17 77.47 0)
 			(effects
@@
 			)
 		)
-		(property "Manufacturer Part" "RV50V47M6X5"
+		(property "Manufacturer Part" "RVT1H470M0607"
 			(at 217.17 77.47 0)
 			(effects
@@
 			)
 		)
-		(property "Manufacturer" "JIERR(捷而瑞)"
+		(property "Manufacturer" "ROQANG(容强)"
 			(at 217.17 77.47 0)
 			(effects
@@
 			)
 		)
-		(property "Supplier Part" "C48971023"
+		(property "Supplier Part" "C72523"
 			(at 217.17 77.47 0)
 			(effects
