File: foc-stepper-driver.kicad_pcb (KiCad board)
At the start: 4 copper layers, 42 x 42 mm, 72 parts, among them CN1 C42391660, CN2 C2839706, CN3 C2839705, CN4 C2839704, J2 TC2030, U1 DRV8962DDWR, U2 TYPE-C 16PLT-H10.0, U3 STM32G431CBT6, U6 AS5047P-ATSM, U7 TPS560430XDBVR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

Commit message: update
Parts:
- added R18: 1k, PCM_Resistor_SMD_AKL:R_0402_1005Metric, F.Cu at (126.1, 85.6)
Connections:
- net /STM32G431CBT6/STM32_CANFD- renamed /STM32G431CBT6/STM32_CANFD_TX
- U3 pad 45: /STM32G431CBT6/STM32_CANFD+ -> Net-(U3-PB8-BOOT0)
- U9 pad 4: /STM32G431CBT6/STM32_CANFD+ -> /STM32G431CBT6/STM32_CANFD_RX
Routing:
- net /STM32G431CBT6/STM32_CANFD+: track 6.43 -> 0.00 mm
- net Net-(U3-PB8-BOOT0): track 0.00 -> 4.01 mm
- net /STM32G431CBT6/STM32_CANFD_RX: track 0.00 -> 2.20 mm

Commit message: update
Routing:
- net GND: track 63.4 -> 63.6 mm, vias 59 -> 60
Changed lines of the file:
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@@
 		(tags "resistor")
 		(property "Reference" "R18"
-			(at 0 -1.3335 90)
+			(at -1.09 1.07 90)
 			(layer "F.SilkS")
 			(effects
 				(font
-					(size 1 1)
-					(thickness 0.15)
+					(size 0.5 0.5)
+					(thickness 0.125)
 				)
 			)
@@
 	)
 	(segment
+		(start 131.56 91.462614)
+		(end 131.3 91.202614)
+		(width 0.2)
+		(layer "F.Cu")
+		(net 1)
+	)
+	(segment
 		(start 136.81 90.77)
 		(end 136.8 90.76)
@@
 	)
 	(segment
+		(start 131.56 91.9)
+		(end 131.56 91.462614)
+		(width 0.2)
+		(layer "F.Cu")
+		(net 1)
+	)
+	(segment
 		(start 136.61 70.46)
 		(end 136.61 71.26)
@@
 	)
 	(segment
-		(start 145.465553 83.978553)
-		(end 145.05 83.563)
-		(width 0.5)
-		(layer "F.Cu")
-		(net 1)
-	)
-	(segment
 		(start 120.269966 87.860034)
 		(end 120.27 87.86)
@@
 	)
 	(via
+		(at 131.3 91.202614)
+		(size 0.6)
+		(drill 0.3)
+		(layers "F.Cu" "B.Cu")
+		(net 1)
+	)
+	(via
 		(at 130.46 79.4)
 		(size 0.6)
@@
 	)
 	(segment
-		(start 131.8 91.2)
-		(end 130.72 91.2)
+		(start 130.46 91.9)
+		(end 130.46 91.05)
 		(width 0.15)
 		(layer "F.Cu")
@@
 	)
 	(segment
-		(start 130.46 91.46)
-		(end 130.46 91.9)
+		(start 130.46 91.05)
+		(end 130.83 90.68)
 		(width 0.15)
 		(layer "F.Cu")
@@
 	)
 	(segment
-		(start 132.42 88.75)
-		(end 132.42 90.58)
+		(start 131.25 90.68)
+		(end 132.42 89.51)
 		(width 0.15)
 		(layer "F.Cu")
@@
 	)
 	(segment
-		(start 132.42 90.58)
-		(end 131.8 91.2)
+		(start 132.42 89.51)
+		(end 132.42 88.75)
 		(width 0.15)
 		(layer "F.Cu")
@@
 	)
 	(segment
-		(start 130.72 91.2)
-		(end 130.46 91.46)
+		(start 130.46 91.9)
+		(end 129.32 91.9)
 		(width 0.15)
 		(layer "F.Cu")
@@
 	)
 	(segment
-		(start 130.46 91.9)
-		(end 129.32 91.9)
+		(start 130.83 90.68)
+		(end 131.25 90.68)
 		(width 0.15)
 		(layer "F.Cu")

Commit message: update
Parts:
- removed R18: 1k, PCM_Resistor_SMD_AKL:R_0402_1005Metric
- removed U9: TCAN3403DRQ1, EasyEDA_Lib:SOP-8_L4.9-W3.9-P1.27-LS6.0-BL
- added C20: 100n, Capacitor_SMD:C_0402_1005Metric, B.Cu at (116.6, 88.4)
- added U4: TCAN1044AVDDFRQ1, EasyEDA_Lib:TSOT-23-8_L2.9-W1.6-P0.65-LS2.8-BR, B.Cu at (119.2, 88.3)
- C16, C22, C23, C27, C29: footprint Capacitor_SMD:C_0402_1005Metric -> Capacitor_SMD:C_0201_0603Metric
- C32: value 10n -> 100n; footprint Capacitor_SMD:C_0402_1005Metric -> Capacitor_SMD:C_0201_0603Metric; moved to B.Cu
- moved C28 13.8 mm to (128.7, 91.2), turned to 180 degrees
- moved C32 4.88 mm to (122.1, 87.4), turned to 0 degrees
- moved C33 0.15 mm to (124.5, 93.1)
Connections:
- U3 pad 26: unconnected-(U3-PB12-Pad26) -> /DRV8962DDWR/DRV8962_nFAULT
- U3 pad 43: /DRV8962DDWR/DRV8962_nFAULT -> /STM32G431CBT6/STM32_CAN_STB
- U3 pad 45: Net-(U3-PB8-BOOT0) -> /STM32G431CBT6/STM32_CANFD_RX
Routing:
- net +5V: track 31.4 -> 58.2 mm
- net /STM32G431CBT6/STM32_CAN_STB: track 0.00 -> 16.3 mm, vias 0 -> 1
- net /STM32G431CBT6/STM32_CANFD_RX: track 2.20 -> 14.9 mm, vias 0 -> 1
- net /DRV8962DDWR/DRV8962_nFAULT: track 34.6 -> 23.8 mm
- net /STM32G431CBT6/STM32_CANFD_TX: track 6.36 -> 17.0 mm, vias 0 -> 1
- net +3.3V: track 29.6 -> 24.6 mm, vias 12 -> 11
- net Net-(U3-PB8-BOOT0): track 4.01 -> 0.00 mm
- net /STM32G431CBT6/CAN_CONN+: track 24.2 -> 21.0 mm, vias 0 -> 1
- net /STM32G431CBT6/CAN_CONN-: track 25.3 -> 22.1 mm, vias 0 -> 1
- net /DRV8962DDWR/DRV8962_MODE: track 24.1 -> 25.7 mm
- net GND: track 63.6 -> 63.4 mm, vias 60 -> 59
Other:
- board text added: "+24V"
- board text added: "A+"
- board text added: "A-"
- board text added: "B+"
- board text added: "B-"
- board text added: "CAN_H"
- board text added: "CAN_L"
- board text added: "GND"
- board text added: "UART_RX"
- board text added: "UART_TX"
- board text added: "USB"

Commit message: update
Parts:
- C13: footprint EasyEDA_Lib:CAP-SMD_BD6.3-L6.6-W6.6-LS7.3-FD -> EasyEDA_Lib:CAP-SMD_BD6.3-L6.6-W6.6-LS7.6-FD
- C16, C22, C23, C27, C29, C32: footprint Capacitor_SMD:C_0201_0603Metric -> Capacitor_SMD:C_0402_1005Metric
- R3: footprint PCM_Resistor_SMD_AKL:R_0402_1005Metric -> Resistor_SMD:R_0805_2012Metric
- R4, R5: footprint Capacitor_SMD:C_0201_0603Metric -> PCM_Resistor_SMD_AKL:R_0402_1005Metric
- R8: footprint PCM_Resistor_SMD_AKL:R_0402_1005Metric -> PCM_Resistor_SMD_AKL:R_0603_1608Metric
- moved R5 1.16 mm to (127.0, 82.9)
- moved C5 0.93 mm to (143.1, 73.6)
- moved R4 0.88 mm to (127.0, 85.0)
- moved R3 0.57 mm to (143.5, 75.2)
- moved R7 0.50 mm to (137.6, 103.1)
- moved R8 0.45 mm to (140.3, 103.1)
- moved C32 0.22 mm to (122.3, 87.3)
- moved C29 0.20 mm to (131.2, 78.7)
- moved C1 0.12 mm to (129.1, 92.7)
- moved C28 0.10 mm to (128.7, 91.3)
- moved C22 0.05 mm to (137.5, 78.7)
Routing:
- net +5V: track 58.2 -> 56.3 mm
- net /STM32G431CBT6/STM32_IC21_SCL: track 1.47 -> 2.70 mm
- net /DRV8962DDWR/DRV8962_nFAULT: track 23.8 -> 24.6 mm
- net +3.3V: track 24.6 -> 25.4 mm, vias 11 -> 12
- net /STM32G431CBT6/STM32_IC21_SDA: track 1.71 -> 2.46 mm
- net Net-(U7-FB): track 2.47 -> 3.19 mm
- net /DRV8962DDWR/DRV8962_DVDD: track 8.42 -> 8.93 mm

Commit message: update
Routing:
- net GND: track 63.8 -> 68.5 mm
- net +3.3V: track 25.4 -> 27.7 mm, vias 12 -> 11
- net +24V: track 29.6 -> 27.7 mm, vias 10 -> 11
- net /DRV8962DDWR/DRV8962_IPROPI1: track 16.8 -> 15.7 mm
