File: POWER.kicad_sch (KiCad schematic)
At the start: 17 parts, among them CN1 C42391660, U7 TPS560430XDBVR, U8 SPX3819M5-L-3-3/TR

Commit message: update
Parts:
- R8: footprint PCM_Resistor_SMD_AKL:R_0402_1005Metric -> PCM_Resistor_SMD_AKL:R_0603_1608Metric
Changed lines of the file:
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@@
 			)
 		)
-		(property "Footprint" "PCM_Resistor_SMD_AKL:R_0402_1005Metric"
+		(property "Footprint" "PCM_Resistor_SMD_AKL:R_0603_1608Metric"
 			(at 144.272 78.74 90)
 			(effects
